File: led.sch (KiCad schematic (older format))
At the start: 115 parts

Commit message: Minor Changes
Parts:
- C10, C11, C12, C13, C14, C15, C16, C17, C18, C19, C20, C21, C22, C23, C24, C9: renamed from C?; footprint (none) -> Capacitors_SMD:C_0805
- LED1, LED10, LED11, LED12, LED13, LED14, LED15, LED16, LED17, LED18, LED19, LED2, LED20, LED21, LED22, LED23, LED24, LED25, LED26, LED27, LED28, LED29, LED3, LED30, LED31, LED32, LED33, LED34, LED35, LED36, LED37, LED38, LED39, LED4, LED40, LED5, LED6, LED7, LED8, LED9: renamed from LED?; footprint (none) -> mx1a:MX1A-led
- LR1, LR10, LR11, LR12, LR13, LR14, LR15, LR16, LR17, LR18, LR19, LR2, LR20, LR21, LR22, LR23, LR24, LR25, LR26, LR27, LR28, LR29, LR3, LR30, LR31, LR32, LR33, LR34, LR35, LR36, LR37, LR38, LR39, LR4, LR40, LR41, LR5, LR6, LR7, LR8, LR9: renamed from LR?; footprint (none) -> Resistors_SMD:R_0805
- Q1: renamed from Q?; footprint (none) -> SI2305:SOT-23
- R4: renamed from R?; footprint (none) -> Resistors_SMD:R_0805
- RGBLED1, RGBLED10, RGBLED11, RGBLED12, RGBLED13, RGBLED14, RGBLED15, RGBLED16, RGBLED2, RGBLED3, RGBLED4, RGBLED5, RGBLED6, RGBLED7, RGBLED8, RGBLED9: renamed from RGBLED?; footprint (none) -> WS2812B:WS2812B
Connections:
- wire segments 434 -> 294

Commit message: ver 0.12
Parts:
- removed C10, C11, C12, C13, C14, C15, C16, C17, C18, C19, C20, C21, C22, C23, C24, C9: 0.1uF, Capacitors_SMD:C_0805, symbol C
- removed RGBLED13, RGBLED14, RGBLED15, RGBLED16: WS2812B, WS2812B:WS2812B, symbol WS2812B
Connections:
- wire segments 294 -> 239

Commit message: a lot of changes
Parts:
- added C10, C11, C12, C13, C14, C15, C16, C17, C18, C19, C9: 100nF, Capacitors_SMD:C_0805, symbol Csmall
Connections:
- wire segments 239 -> 282

Commit message: minor changes & update gerber files
Parts:
- added C20: 100nF, Capacitors_SMD:C_0805, symbol Csmall
Connections:
- wire segments 282 -> 284
Changed lines of the file:
@@
 	3950 8650 3950 9100
 Wire Wire Line
-	3950 8950 16000 8950
+	3950 8950 16650 8950
 Wire Wire Line
 	5000 8950 5000 8650
@@
 	14900 8000 14900 7650
 Connection ~ 14900 7650
+$Comp
+L Csmall C20
+U 1 1 57780F5C
+P 16250 8100
+F 0 "C20" H 16275 8150 30  0000 L CNN
+F 1 "100nF" H 16275 8050 30  0000 L CNN
+F 2 "Capacitors_SMD:C_0805" H 16250 8100 60  0001 C CNN
+F 3 "" H 16250 8100 60  0000 C CNN
+	1    16250 8100
+	1    0    0    -1
+$EndComp
+Connection ~ 16000 8950
+Wire Wire Line
+	16250 8200 16250 8950
+Connection ~ 16250 8950
+Wire Wire Line
+	16250 8000 16250 7650
+Connection ~ 16250 7650
 $EndSCHEMATC
