File: keyboard.sch (KiCad schematic (older format))
At the start: 74 parts, among them IC1 ATMEGA32U4, J1 MINI, P1 MISO, P10 ROW4, P18 LR1, P19 LR2, P2 Vcc, P20 LR3, P200 GND, P201 GND, P202 GND, P203 GND, P21 LR4, P23 LC1, P24 LC2, P25 LC3, P26 LC4, P27 LC5, P28 LC6, P29 LC7, P3 SCK, P30 LC8, P31 LC9, P32 LC10, P33 LC11, P34 LC12, P35 LGND, P36 LVcc, P37 Vcc, P38 GPIO0, P39 GPIO1, P4 MOSI, P40 GPIO2, P41 GPIO3, P42 GPIO4(SS), P43 GPIO5(SCK), P44 GPIO6(MOSI), P45 GPIO7(SCL), P46 GPIO8(SDA), P47 GND, P5 RES, P6 GND, P7 ROW1, P8 ROW2, P9 ROW3, X1 ASX3F

Commit message: Change the cyrstal footprint / correct two wrong diode directions
Parts:
- removed X1: ASX3F, symbol ASX4
- added X1: CRYSTAL, symbol CRYSTAL
Connections:
- wire segments 170 -> 168
Changed lines of the file:
@@
-EESchema Schematic File Version 2  date 11/23/2013 1:19:47 PM
+EESchema Schematic File Version 2
 LIBS:power
 LIBS:mx1a-simple
@@
 LIBS:usb_ports
 LIBS:keyboard-cache
-EELAYER 27 0
+EELAYER 25 0
 EELAYER END
 $Descr A4 11693 8268
@@
 $EndComp
 $Comp
-L GND #PWR03
-U 1 1 4F08176B
-P 2100 4450
-F 0 "#PWR03" H 2100 4450 30  0001 C CNN
-F 1 "GND" H 2100 4380 30  0001 C CNN
-F 2 "" H 2100 4450 60  0001 C CNN
-F 3 "" H 2100 4450 60  0001 C CNN
-	1    2100 4450
-	1    0    0    -1
-$EndComp
-$Comp
-L GND #PWR04
-U 1 1 4F081769
-P 1900 4450
-F 0 "#PWR04" H 1900 4450 30  0001 C CNN
-F 1 "GND" H 1900 4380 30  0001 C CNN
-F 2 "" H 1900 4450 60  0001 C CNN
-F 3 "" H 1900 4450 60  0001 C CNN
-	1    1900 4450
-	1    0    0    -1
-$EndComp
-$Comp
-L ASX4 X1
-U 1 1 4F081730
-P 2000 4000
-F 0 "X1" H 2000 3800 60  0000 C CNN
-F 1 "ASX3F" H 2000 4200 60  0000 C CNN
-F 2 "" H 2000 4000 60  0001 C CNN
-F 3 "" H 2000 4000 60  0001 C CNN
-F 4 "YIC" H 2000 4000 60  0001 C CNN "Vendor"
-F 5 "16.00M-SMDXT324" H 2000 4000 60  0001 C CNN "Product"
-F 6 "TME" H 2000 4000 60  0001 C CNN "Supplier"
-F 7 "16.00M-SMDXT324" H 2000 4000 60  0001 C CNN "Supplier Symbol"
-	1    2000 4000
-	1    0    0    -1
-$EndComp
-$Comp
-L VCC #PWR05
+L VCC #PWR03
 U 1 1 4ED6BD35
 P 4700 1050
-F 0 "#PWR05" H 4700 1150 30  0001 C CNN
+F 0 "#PWR03" H 4700 1150 30  0001 C CNN
 F 1 "VCC" H 4700 1150 30  0000 C CNN
 F 2 "" H 4700 1050 60  0001 C CNN
@@
 $EndComp
 $Comp
-L GND #PWR06
+L GND #PWR04
 U 1 1 4ED6BD03
 P 4700 1850
-F 0 "#PWR06" H 4700 1850 30  0001 C CNN
+F 0 "#PWR04" H 4700 1850 30  0001 C CNN
 F 1 "GND" H 4700 1780 30  0001 C CNN
 F 2 "" H 4700 1850 60  0001 C CNN
@@
 	3000 1200 3100 1300
 $Comp
-L GND #PWR07
+L GND #PWR05
 U 1 1 4ED6BB30
 P 800 3500
-F 0 "#PWR07" H 800 3500 30  0001 C CNN
+F 0 "#PWR05" H 800 3500 30  0001 C CNN
 F 1 "GND" H 800 3430 30  0001 C CNN
 F 2 "" H 800 3500 60  0001 C CNN
@@
 $EndComp
 $Comp
-L VCC #PWR08
+L VCC #PWR06
 U 1 1 4ED6BA8E
 P 2550 750
-F 0 "#PWR08" H 2550 850 30  0001 C CNN
+F 0 "#PWR06" H 2550 850 30  0001 C CNN
 F 1 "VCC" H 2550 850 30  0000 C CNN
 F 2 "" H 2550 750 60  0001 C CNN
@@
 $EndComp
 $Comp
-L GND #PWR09
+L GND #PWR07
 U 1 1 4ED6AF1D
 P 5100 7400
-F 0 "#PWR09" H 5100 7400 30  0001 C CNN
+F 0 "#PWR07" H 5100 7400 30  0001 C CNN
 F 1 "GND" H 5100 7330 30  0001 C CNN
 F 2 "" H 5100 7400 60  0001 C CNN
@@
 $EndComp
 $Comp
-L GND #PWR010
+L GND #PWR08
 U 1 1 4ED6A667
 P 2600 7350
-F 0 "#PWR010" H 2600 7350 30  0001 C CNN
+F 0 "#PWR08" H 2600 7350 30  0001 C CNN
 F 1 "GND" H 2600 7280 30  0001 C CNN
 F 2 "" H 2600 7350 60  0001 C CNN
@@
 $EndComp
 $Comp
-L GND #PWR011
+L GND #PWR09
 U 1 1 4ED6A5D7
 P 2350 7350
-F 0 "#PWR011" H 2350 7350 30  0001 C CNN
+F 0 "#PWR09" H 2350 7350 30  0001 C CNN
 F 1 "GND" H 2350 7280 30  0001 C CNN
 F 2 "" H 2350 7350 60  0001 C CNN
@@
 $EndComp
 $Comp
-L GND #PWR012
+L GND #PWR010
 U 1 1 4ED6A418
 P 1500 6250
-F 0 "#PWR012" H 1500 6250 30  0001 C CNN
+F 0 "#PWR010" H 1500 6250 30  0001 C CNN
 F 1 "GND" H 1500 6180 30  0001 C CNN
 F 2 "" H 1500 6250 60  0001 C CNN
@@
 $EndComp
 $Comp
-L VCC #PWR013
+L VCC #PWR011
 U 1 1 4EB30C92
 P 3550 2250
-F 0 "#PWR013" H 3550 2350 30  0001 C CNN
+F 0 "#PWR011" H 3550 2350 30  0001 C CNN
 F 1 "VCC" H 3550 2350 30  0000 C CNN
 F 2 "" H 3550 2250 60  0001 C CNN
@@
 $EndComp
 $Comp
-L VCC #PWR014
+L VCC #PWR012
 U 1 1 4EB30C91
 P 3650 2250
-F 0 "#PWR014" H 3650 2350 30  0001 C CNN
+F 0 "#PWR012" H 3650 2350 30  0001 C CNN
 F 1 "VCC" H 3650 2350 30  0000 C CNN
 F 2 "" H 3650 2250 60  0001 C CNN
@@
 $EndComp
 $Comp
-L VCC #PWR015
+L VCC #PWR013
 U 1 1 4EB30C90
 P 3850 2250
-F 0 "#PWR015" H 3850 2350 30  0001 C CNN
+F 0 "#PWR013" H 3850 2350 30  0001 C CNN
 F 1 "VCC" H 3850 2350 30  0000 C CNN
 F 2 "" H 3850 2250 60  0001 C CNN
@@
 $EndComp
 $Comp
-L VCC #PWR016
+L VCC #PWR014
 U 1 1 4EB30C8B
 P 3950 2250
-F 0 "#PWR016" H 3950 2350 30  0001 C CNN
+F 0 "#PWR014" H 3950 2350 30  0001 C CNN
 F 1 "VCC" H 3950 2350 30  0000 C CNN
 F 2 "" H 3950 2250 60  0001 C CNN
@@
 	5200 4050 5300 4150
 $Comp
-L GND #PWR017
+L GND #PWR015
 U 1 1 4EB2CF09
 P 1100 1900
-F 0 "#PWR017" H 1100 1900 30  0001 C CNN
+F 0 "#PWR015" H 1100 1900 30  0001 C CNN
 F 1 "GND" H 1100 1830 30  0001 C CNN
 F 2 "" H 1100 1900 60  0001 C CNN
@@
 $EndComp
 $Comp
-L VCC #PWR018
+L VCC #PWR016
 U 1 1 4EB2CED6
 P 1100 750
-F 0 "#PWR018" H 1100 850 30  0001 C CNN
+F 0 "#PWR016" H 1100 850 30  0001 C CNN
 F 1 "VCC" H 1100 850 30  0000 C CNN
 F 2 "" H 1100 750 60  0001 C CNN
@@
 $EndComp
 $Comp
-L GND #PWR019
+L GND #PWR017
 U 1 1 4E99C40C
 P 3900 7350
-F 0 "#PWR019" H 3900 7350 30  0001 C CNN
+F 0 "#PWR017" H 3900 7350 30  0001 C CNN
 F 1 "GND" H 3900 7280 30  0001 C CNN
 F 2 "" H 3900 7350 60  0001 C CNN
@@
 $EndComp
 $Comp
-L GND #PWR020
+L GND #PWR018
 U 1 1 4E99C40B
 P 3800 7350
-F 0 "#PWR020" H 3800 7350 30  0001 C CNN
+F 0 "#PWR018" H 3800 7350 30  0001 C CNN
 F 1 "GND" H 3800 7280 30  0001 C CNN
 F 2 "" H 3800 7350 60  0001 C CNN
@@
 $EndComp
 $Comp
-L GND #PWR021
+L GND #PWR019
 U 1 1 4E99C407
 P 3700 7350
-F 0 "#PWR021" H 3700 7350 30  0001 C CNN
+F 0 "#PWR019" H 3700 7350 30  0001 C CNN
 F 1 "GND" H 3700 7280 30  0001 C CNN
 F 2 "" H 3700 7350 60  0001 C CNN
@@
 $EndComp
 $Comp
-L GND #PWR022
+L GND #PWR020
 U 1 1 4E99C403
 P 3600 7350
-F 0 "#PWR022" H 3600 7350 30  0001 C CNN
+F 0 "#PWR020" H 3600 7350 30  0001 C CNN
 F 1 "GND" H 3600 7280 30  0001 C CNN
 F 2 "" H 3600 7350 60  0001 C CNN
@@
 $EndComp
 $Comp
-L GND #PWR023
+L GND #PWR021
 U 1 1 4E99B659
-P 1550 4750
-F 0 "#PWR023" H 1550 4750 30  0001 C CNN
-F 1 "GND" H 1550 4680 30  0001 C CNN
-F 2 "" H 1550 4750 60  0001 C CNN
-F 3 "" H 1550 4750 60  0001 C CNN
-	1    1550 4750
-	1    0    0    -1
-$EndComp
-$Comp
-L GND #PWR024
-U 1 1 4E99B657
-P 2450 4750
-F 0 "#PWR024" H 2450 4750 30  0001 C CNN
-F 1 "GND" H 2450 4680 30  0001 C CNN
-F 2 "" H 2450 4750 60  0001 C CNN
-F 3 "" H 2450 4750 60  0001 C CNN
-	1    2450 4750
-	1    0    0    -1
-$EndComp
-$Comp
-L GND #PWR025
-U 1 1 4E99B655
-P 2450 4750
-F 0 "#PWR025" H 2450 4750 30  0001 C CNN
-F 1 "GND" H 2450 4680 30  0001 C CNN
-F 2 "" H 2450 4750 60  0001 C CNN
-F 3 "" H 2450 4750 60  0001 C CNN
-	1    2450 4750
+P 1950 4750
+F 0 "#PWR021" H 1950 4750 30  0001 C CNN
+F 1 "GND" H 1950 4680 30  0001 C CNN
+F 2 "" H 1950 4750 60  0001 C CNN
+F 3 "" H 1950 4750 60  0001 C CNN
+	1    1950 4750
 	1    0    0    -1
 $EndComp
@@
 GPIO3
 $Comp
-L VCC #PWR026
+L VCC #PWR022
 U 1 1 516C9166
 P 10850 3050
-F 0 "#PWR026" H 10850 3150 30  0001 C CNN
+F 0 "#PWR022" H 10850 3150 30  0001 C CNN
 F 1 "VCC" H 10850 3150 30  0000 C CNN
 F 2 "" H 10850 3050 60  0001 C CNN
@@
 GPIO3
 $Comp
-L VCC #PWR027
+L VCC #PWR023
 U 1 1 51CCBD4D
 P 9350 750
-F 0 "#PWR027" H 9350 850 30  0001 C CNN
+F 0 "#PWR023" H 9350 850 30  0001 C CNN
 F 1 "VCC" H 9350 850 30  0000 C CNN
 F 2 "" H 9350 750 60  0001 C CNN
@@
 $EndComp
 $Comp
-L GND #PWR028
+L GND #PWR024
 U 1 1 51CCCE51
 P 9350 2150
-F 0 "#PWR028" H 9350 2150 30  0001 C CNN
+F 0 "#PWR024" H 9350 2150 30  0001 C CNN
 F 1 "GND" H 9350 2080 30  0001 C CNN
 F 2 "" H 9350 2150 60  0001 C CNN
@@
 $EndComp
 $Comp
-L GND #PWR029
+L GND #PWR025
 U 1 1 523205C7
 P 5650 3050
-F 0 "#PWR029" H 5650 3050 30  0001 C CNN
+F 0 "#PWR025" H 5650 3050 30  0001 C CNN
 F 1 "GND" H 5650 2980 30  0001 C CNN
 F 2 "" H 5650 3050 60  0001 C CNN
@@
 	800  3500 800  3200
 Wire Wire Line
-	2100 4250 2100 4450
-Wire Wire Line
-	2250 4000 2750 4000
+	2300 4000 2750 4000
 Wire Wire Line
 	4700 1300 4700 1050
@@
 Wire Wire Line
 	3600 6900 3600 7350
-Wire Wire Line
-	2450 4550 2450 4750
 Connection ~ 2450 4000
 Wire Wire Line
@@
 Connection ~ 1550 4000
 Wire Wire Line
-	1550 4550 1550 4750
-Wire Wire Line
 	3700 6900 3700 7350
 Wire Wire Line
@@
 Wire Wire Line
 	4700 1850 4700 1500
-Wire Wire Line
-	1750 4000 1550 4000
-Wire Wire Line
-	1900 4250 1900 4450
 Wire Wire Line
 	4750 5050 6100 5050
@@
 $EndComp
 $Comp
-L VCC #PWR030
+L VCC #PWR026
 U 1 1 528FE3F1
 P 8150 2400
-F 0 "#PWR030" H 8150 2500 30  0001 C CNN
+F 0 "#PWR026" H 8150 2500 30  0001 C CNN
 F 1 "VCC" H 8150 2500 30  0000 C CNN
 F 2 "" H 8150 2400 60  0001 C CNN
@@
 $EndComp
 $Comp
-L GND #PWR031
+L GND #PWR027
 U 1 1 528FE3F7
 P 8150 2300
-F 0 "#PWR031" H 8150 2300 30  0001 C CNN
+F 0 "#PWR027" H 8150 2300 30  0001 C CNN
 F 1 "GND" H 8150 2230 30  0001 C CNN
 F 2 "" H 8150 2300 60  0001 C CNN
@@
 Text Notes 9600 3150 0    60   ~ 0
 SW01  LED (ESCAPE)\n
+$Comp
+L CRYSTAL X1
+U 1 1 57381836
+P 2000 4000
+F 0 "X1" H 2000 4150 60  0000 C CNN
+F 1 "CRYSTAL" H 2000 3850 60  0000 C CNN
+F 2 "" H 2000 4000 60  0000 C CNN
+F 3 "" H 2000 4000 60  0000 C CNN
+	1    2000 4000
+	1    0    0    -1
+$EndComp
+Wire Wire Line
+	1550 4000 1700 4000
+Wire Wire Line
+	2450 4550 1550 4550
+Wire Wire Line
+	1950 4550 1950 4750
+Connection ~ 1950 4550
 $EndSCHEMATC

Commit message: Change the footprint of MiniUSB
Connections:
- net labels added: D+, D-
Other:
- note added: "FN LED\n"
- moved on the sheet: DF3, R12
Changed lines of the file:
@@
 	1    0    0    -1
 $EndComp
-Text Label 9150 3350 0    50   ~ 0
+Text Label 9100 4500 0    50   ~ 0
 GPIO1
 $Comp
 L LED DF3
 U 1 1 5179BCCC
-P 10450 3350
-F 0 "DF3" H 9850 3350 50  0000 L CNN
-F 1 "LED" H 10600 3250 50  0000 C CNN
-F 2 "" H 10450 3350 60  0001 C CNN
-F 3 "" H 10450 3350 60  0001 C CNN
-	1    10450 3350
+P 10450 4500
+F 0 "DF3" H 9850 4500 50  0000 L CNN
+F 1 "LED" H 10600 4400 50  0000 C CNN
+F 2 "" H 10450 4500 60  0001 C CNN
+F 3 "" H 10450 4500 60  0001 C CNN
+	1    10450 4500
 	-1   0    0    1
 $EndComp
@@
 L R R12
 U 1 1 5179BCD2
-P 9850 3350
-F 0 "R12" V 9930 3350 50  0000 C CNN
-F 1 "R" V 9850 3350 50  0000 C CNN
-F 2 "" H 9850 3350 60  0001 C CNN
-F 3 "" H 9850 3350 60  0001 C CNN
-	1    9850 3350
+P 9850 4500
+F 0 "R12" V 9930 4500 50  0000 C CNN
+F 1 "R" V 9850 4500 50  0000 C CNN
+F 2 "" H 9850 4500 60  0001 C CNN
+F 3 "" H 9850 4500 60  0001 C CNN
+	1    9850 4500
 	0    -1   -1   0
 $EndComp
 Entry Wire Line
-	8950 3450 9050 3350
+	8950 4600 9050 4500
 $Sheet
 S 6550 700  1250 1900
@@
 	8950 6350 8950 6450
 Wire Wire Line
-	9050 3350 9600 3350
-Wire Wire Line
-	10100 3350 10250 3350
-Wire Wire Line
-	10650 3350 10850 3350
-Connection ~ 10850 3350
+	9050 4500 9600 4500
+Wire Wire Line
+	10100 4500 10250 4500
+Wire Wire Line
+	10850 4500 10650 4500
+Connection ~ 10850 4500
 Wire Bus Line
 	3000 900  5300 900
@@
 	6550 6500 6200 6500
 Wire Bus Line
-	6200 6500 6200 3300
+	6200 3300 6200 6500
 Wire Bus Line
 	6550 2950 6550 6500
@@
 Text Notes 9750 5050 0    60   ~ 0
 WASD Cluster LEDs\n
-Text Notes 9600 3150 0    60   ~ 0
+Text Notes 9500 4350 0    60   ~ 0
 SW01  LED (ESCAPE)\n
 $Comp
@@
 	1550 4000 1700 4000
 Wire Wire Line
-	2450 4550 1550 4550
+	1550 4550 2450 4550
 Wire Wire Line
 	1950 4550 1950 4750
 Connection ~ 1950 4550
+Text Notes 9900 4700 0    60   ~ 0
+FN LED\n
+Text Label 1450 5750 0    60   ~ 0
+D-
+Text Label 1450 5850 0    60   ~ 0
+D+
 $EndSCHEMATC

Commit message: Rebuild the project using latest kicad
Rebuild the project using latest kicad, leaving eschematic and pcb
unfinished
Parts:
- removed C4, C5, C6, C7: 100n, symbol C
- removed C8: 1u, symbol C
- removed DF3, DW1, DW2, DW3, DW4: LED, symbol LED
- removed H1, H2, H3, H4, H5: HOLE, ~, symbol ANYTHING
- removed J1: MINI, symbol USBMINI_B05
- removed P1: MISO, symbol CONN_1
- removed P10: ROW4, symbol CONN_1
- removed P18: LR1, symbol CONN_1
- removed P19: LR2, symbol CONN_1
- removed P2, P37: Vcc, symbol CONN_1
- removed P20: LR3, symbol CONN_1
- removed P200, P201, P202, P203, P47, P6: GND, symbol CONN_1
- removed P21: LR4, symbol CONN_1
- removed P23: LC1, symbol CONN_1
- removed P24: LC2, symbol CONN_1
- removed P25: LC3, symbol CONN_1
- removed P26: LC4, symbol CONN_1
- removed P27: LC5, symbol CONN_1
- removed P28: LC6, symbol CONN_1
- removed P29: LC7, symbol CONN_1
- removed P3: SCK, symbol CONN_1
- removed P30: LC8, symbol CONN_1
- removed P31: LC9, symbol CONN_1
- removed P32: LC10, symbol CONN_1
- removed P33: LC11, symbol CONN_1
- removed P34: LC12, symbol CONN_1
- removed P35: LGND, symbol CONN_1
- removed P36: LVcc, symbol CONN_1
- removed P38: GPIO0, symbol CONN_1
- removed P39: GPIO1, symbol CONN_1
- removed P4: MOSI, symbol CONN_1
- removed P40: GPIO2, symbol CONN_1
- removed P41: GPIO3, symbol CONN_1
- removed P42: GPIO4(SS), symbol CONN_1
- removed P43: GPIO5(SCK), symbol CONN_1
- removed P44: GPIO6(MOSI), symbol CONN_1
- removed P45: GPIO7(SCL), symbol CONN_1
- removed P46: GPIO8(SDA), symbol CONN_1
- removed P5: RES, symbol CONN_1
- removed P7: ROW1, symbol CONN_1
- removed P8: ROW2, symbol CONN_1
- removed P9: ROW3, symbol CONN_1
- removed R12, RW1, RW2, RW3, RW4: R, symbol R
- removed R3: 10k, symbol R
- removed X1: CRYSTAL, symbol CRYSTAL
- added J?: USBMINI_B05, symbol USBMINI_B05
- added R?: R, symbol R
- added X?: CRYSTAL, symbol CRYSTAL
- C1, C2: value 22p -> 22pF; Product CL21C220JBANNNC -> (none); Supplier TME -> (none); Supplier Symbol CL21C220JBANNNC -> (none); Vendor Samsung -> (none)
- C3: value 1u -> 1uF; Product CL21B105KAFNNNE -> (none); Supplier TME -> (none); Supplier Symbol CL21B105KAFNNNE -> (none); Vendor Samsung -> (none)
- IC1: Product ATmega32U4-AU -> (none); Supplier DigiKey -> (none); Supplier Symbol ATMEGA32U4-AU-ND -> (none); Vendor Atmel -> (none)
- R1, R2: value 22 -> 22R; Product CRCW080522R0JNTABC -> (none); Supplier TME -> (none); Supplier Symbol CRCW080522R0JNTABC -> (none); Vendor Vishay -> (none)
- R5: value 10k -> 10K; Product CRCW080510K0JNTABC -> (none); Supplier TME -> (none); Supplier Symbol CRCW080510K0JNTABC -> (none); Vendor Vishay -> (none)
- S0: Product TACTB-64K-F -> (none); Supplier TME -> (none); Supplier Symbol TACTB-64K-F -> (none); Vendor Ninigi -> (none)
Connections:
- net labels removed: D+, D-, GPIO0, GPIO1, GPIO2, GPIO3, GPIO4, GPIO5, GPIO6, GPIO7, GPIO8, MISO, MOSI, SCK, SCL, SDA, SS, caps, col1, col10, col11, col2, col3, col4, col5, col6, col7, col8, col9, row1, row2, row3, row4, ~RES~
- wire segments 168 -> 46
- no-connect marks 4 -> 2
Other:
- note removed: "Expansion\nconnector \n(right)"
- note removed: "FN LED\n"
- note removed: "Ground Pins"
- note removed: "ISP Pins"
- note removed: "LED Matrix\n(top)"
- note removed: "Mounting\nHoles"
- note removed: "PWM"
- note removed: "SW01 LED (ESCAPE)\n"
- note removed: "WASD Cluster LEDs\n"

Commit message: Final touches on schematic
Parts:
- added P1, P2, P3 (x2), P4, P5 (x2), P6, P7, P8: CONN_1, symbol CONN_1
Connections:
- net GND: now also P4.1
- net VCC: now also P2.1
- net Backlight: now reaches IC1.1 ((INT6/AIN0)PE6)
- net GPIO0: now reaches IC1.10 ((PDI/PCINT2/MOSI)PB2)
- net GPIO0: now also P3.1, P7.1, P8.1
- net Col6: now reaches IC1.11 ((PDO/PCINT3/MISO)PB3)
- net Col6: now also P1.1
- net Col10: now reaches IC1.12 ((PCINT7/OC0A/OC1C/~RTS~)PB7)
- net ~Res: now reaches IC1.13 (~RESET~), R5.2, S0.3
- net ~Res: now also P5.1
- net GPIO4: now reaches IC1.18 ((OC0B/SCL/INT0)PD0)
- net GPIO3: now reaches IC1.19 ((SDA/INT1)PD1)
- net GPIO3: now also P5.1
- net Row0: now reaches IC1.20 ((RXD1/INT2)PD2)
- net Row1: now reaches IC1.21 ((TXD1/INT3)PD3)
- net Row3: now reaches IC1.22 ((XCK1/~CTS~)PD5)
- net Row2: now reaches IC1.25 ((ICP1/ADC8)PD4)
- net WASD: now reaches IC1.26 ((T1/~OC4D~/ADC9)PD6)
- net ESC: now reaches IC1.27 ((T0/OC4D/ADC10)PD7)
- net Col7: now reaches IC1.28 ((PCINT4/ADC11)PB4)
- net Col8: now reaches IC1.29 ((PCINT5/OC1A/~OC4B~/ADC12)PB5)
- net Col9: now reaches IC1.30 ((PCINT6/OC1B/OC4B/ADC13)PB6)
- net Caps: now reaches IC1.31 ((OC3A/~OC4A~)PC6)
- net Bottom: now reaches IC1.32 ((ICP3/CLK0/OC4A)PC7)
- net Col5: now reaches IC1.36 ((ADC7/TDI)PF7)
- net Col4: now reaches IC1.37 ((ADC6/TDO)PF6)
- net Col3: now reaches IC1.38 ((ADC5/TMS)PF5)
- net Col2: now reaches IC1.39 ((ADC4/TCK)PF4)
- net Col1: now reaches IC1.40 ((ADC1)PF1)
- net Col0: now reaches IC1.41 ((ADC0)PF0)
- net GPIO2: now reaches IC1.8 ((SS/PCINT0)PB0)
- net GPIO2: now also P6.1
- net SCK: now reaches IC1.9 ((PCINT1/SCLK)PB1)
- net SCK: now also P3.1
Other:
- moved on the sheet: R5, R?

Commit message: Final touches on schematic
Parts:
- removed P1, P2, P3 (x2), P4, P5 (x2), P6, P7, P8: CONN_1, symbol CONN_1
- added C4, C5, C6, C7: 100nF, symbol C
- added C8: 1uF, symbol C
- added P1: ISP, symbol CONN_3X2
- added P2: GPIO Port, symbol CONN_4
- R3: renamed from R?; value R -> 10K
Connections:
- net Col6: now also P1.1
- net GND: now also C4.2, C5.2, C6.2, C7.2, C8.2, P1.6
- net GPIO0: now also P1.4, P2.3 (P3), P2.4 (P4)
- net GPIO2: now also P2.2 (P2)
- net GPIO3: now also P2.1 (P1)
- net SCK: now also P1.3
- net VCC: now also C4.1, C5.1, C6.1, C7.1, C8.1, P1.2
- net ~Res: now also P1.5
- no-connect marks 2 -> 4
