File: keyboard.sch (KiCad schematic (older format))
At the start: 18 parts, among them IC1 ATMEGA32U4, P1 ISP, P2 GPIO Port

Commit message: Minor Changes
Parts:
- C1, C2, C3, C4, C5, C6, C7, C8: footprint (none) -> Capacitors_SMD:C_0805
- IC1: footprint TQFP44 -> tqfp:TQFP44
- J1: renamed from J?; footprint (none) -> USB:DX_USB
- P1: footprint (none) -> Socket_Strips:Socket_Strip_Straight_2x03
- P2: footprint (none) -> Socket_Strips:Socket_Strip_Straight_1x04
- R1, R2, R3, R5: footprint (none) -> Resistors_SMD:R_0805
- S0: footprint switch-tact-DTSM-6 -> switch:DTSM-6
- X1: renamed from X?; footprint (none) -> Crystals:Crystal_HC49-U_Vertical
Changed lines of the file:
@@
 F 0 "IC1" H 4250 6180 50  0000 L BNN
 F 1 "ATMEGA32U4" H 5300 2450 50  0000 L BNN
-F 2 "TQFP44" H 5550 2375 50  0001 C CNN
+F 2 "tqfp:TQFP44" H 5550 2375 50  0001 C CNN
 F 3 "" H 5050 4350 60  0000 C CNN
 	1    5050 4350
@@
 $EndComp
 $Comp
-L CRYSTAL X?
+L CRYSTAL X1
 U 1 1 573FEA9B
 P 3550 3450
-F 0 "X?" H 3550 3600 60  0000 C CNN
+F 0 "X1" H 3550 3600 60  0000 C CNN
 F 1 "CRYSTAL" H 3550 3300 60  0000 C CNN
-F 2 "" H 3550 3450 60  0000 C CNN
+F 2 "Crystals:Crystal_HC49-U_Vertical" H 3550 3450 60  0001 C CNN
 F 3 "" H 3550 3450 60  0000 C CNN
 	1    3550 3450
@@
 F 0 "C1" H 3000 3900 50  0000 L CNN
 F 1 "22pF" H 3000 3700 50  0000 L CNN
-F 2 "" H 2950 3800 60  0000 C CNN
+F 2 "Capacitors_SMD:C_0805" H 2950 3800 60  0001 C CNN
 F 3 "" H 2950 3800 60  0000 C CNN
 	1    2950 3800
@@
 F 0 "C2" H 4050 3900 50  0000 L CNN
 F 1 "22pF" H 4050 3700 50  0000 L CNN
-F 2 "" H 4000 3800 60  0000 C CNN
+F 2 "Capacitors_SMD:C_0805" H 4000 3800 60  0001 C CNN
 F 3 "" H 4000 3800 60  0000 C CNN
 	1    4000 3800
@@
 F 0 "S0" V 2565 2550 50  0000 L BNN
 F 1 "DTSM-6" V 2665 2775 50  0000 L BNN
-F 2 "switch-tact-DTSM-6" H 2850 2800 50  0001 C CNN
+F 2 "switch:DTSM-6" H 2850 2800 50  0001 C CNN
 F 3 "" H 2850 2650 60  0000 C CNN
 	1    2850 2650
@@
 F 0 "R5" V 3780 1300 50  0000 C CNN
 F 1 "10K" V 3700 1300 50  0000 C CNN
-F 2 "" H 3700 1300 60  0000 C CNN
+F 2 "Resistors_SMD:R_0805" H 3700 1300 60  0001 C CNN
 F 3 "" H 3700 1300 60  0000 C CNN
 	1    3700 1300
@@
 F 0 "R1" V 3530 5200 50  0000 C CNN
 F 1 "22R" V 3450 5200 50  0000 C CNN
-F 2 "" H 3450 5200 60  0000 C CNN
+F 2 "Resistors_SMD:R_0805" H 3450 5200 60  0001 C CNN
 F 3 "" H 3450 5200 60  0000 C CNN
 	1    3450 5200
@@
 F 0 "R2" V 3530 5300 50  0000 C CNN
 F 1 "22R" V 3450 5300 50  0000 C CNN
-F 2 "" H 3450 5300 60  0000 C CNN
+F 2 "Resistors_SMD:R_0805" H 3450 5300 60  0001 C CNN
 F 3 "" H 3450 5300 60  0000 C CNN
 	1    3450 5300
@@
 $EndComp
 $Comp
-L USBMINI_B05 J?
+L USBMINI_B05 J1
 U 1 1 5740162B
 P 2700 5300
-F 0 "J?" H 2625 5600 60  0000 C CNN
+F 0 "J1" H 2625 5600 60  0000 C CNN
 F 1 "USBMINI_B05" H 2650 4950 60  0001 C CNN
-F 2 "" H 2700 5300 60  0000 C CNN
+F 2 "USB:DX_USB" H 2700 5300 60  0001 C CNN
 F 3 "" H 2700 5300 60  0000 C CNN
 	1    2700 5300
@@
 F 0 "C3" H 3800 6050 50  0000 L CNN
 F 1 "1uF" H 3800 5850 50  0000 L CNN
-F 2 "" H 3750 5950 60  0000 C CNN
+F 2 "Capacitors_SMD:C_0805" H 3750 5950 60  0001 C CNN
 F 3 "" H 3750 5950 60  0000 C CNN
 	1    3750 5950
@@
 F 0 "R3" V 6230 6200 50  0000 C CNN
 F 1 "10K" V 6150 6200 50  0000 C CNN
-F 2 "" H 6150 6200 60  0000 C CNN
+F 2 "Resistors_SMD:R_0805" H 6150 6200 60  0001 C CNN
 F 3 "" H 6150 6200 60  0000 C CNN
 	1    6150 6200
@@
 	4050 3050 2950 3050
 Wire Wire Line
-	2950 3050 2950 3450
-Wire Wire Line
-	2950 3450 2950 3600
+	2950 3050 2950 3600
 Wire Wire Line
 	2950 3450 3250 3450
 Wire Wire Line
-	3850 3450 4000 3450
-Wire Wire Line
-	4000 3450 4050 3450
+	3850 3450 4050 3450
 Connection ~ 2950 3450
 Wire Wire Line
@@
 	2950 4000 2950 4050
 Wire Wire Line
-	2950 4050 3500 4050
-Wire Wire Line
-	3500 4050 4000 4050
+	2950 4050 4000 4050
 Wire Wire Line
 	4000 4050 4000 4000
@@
 	2400 2650 2650 2650
 Wire Wire Line
-	3050 2650 3700 2650
-Wire Wire Line
-	3700 2650 4050 2650
+	3050 2650 4050 2650
 Connection ~ 3700 2650
 Wire Wire Line
@@
 	3900 5500 4050 5500
 Wire Wire Line
-	3900 4850 3900 5000
-Wire Wire Line
-	3900 5000 3900 5500
+	3900 4850 3900 5500
 Wire Wire Line
 	4050 5000 3900 5000
@@
 	6600 5100 6700 5200
 Wire Bus Line
-	6700 2550 6700 3000
+	6700 2550 6700 6100
 Wire Bus Line
-	6700 3000 6700 3100
+	6700 6100 8150 6100
 Wire Bus Line
-	6700 3100 6700 3200
-Wire Bus Line
-	6700 3200 6700 3300
-Wire Bus Line
-	6700 3300 6700 3400
-Wire Bus Line
-	6700 3400 6700 3500
-Wire Bus Line
-	6700 3500 6700 3600
-Wire Bus Line
-	6700 3600 6700 3700
-Wire Bus Line
-	6700 3700 6700 3900
-Wire Bus Line
-	6700 3900 6700 4000
-Wire Bus Line
-	6700 4000 6700 4200
-Wire Bus Line
-	6700 4200 6700 4300
-Wire Bus Line
-	6700 4300 6700 4400
-Wire Bus Line
-	6700 4400 6700 4500
-Wire Bus Line
-	6700 4500 6700 4600
-Wire Bus Line
-	6700 4600 6700 4700
-Wire Bus Line
-	6700 4700 6700 4800
-Wire Bus Line
-	6700 4800 6700 4900
-Wire Bus Line
-	6700 4900 6700 5200
-Wire Bus Line
-	6700 5200 6700 5400
-Wire Bus Line
-	6700 5400 6700 5500
-Wire Bus Line
-	6700 5500 6700 5600
-Wire Bus Line
-	6700 5600 6700 5700
-Wire Bus Line
-	6700 5700 6700 5800
-Wire Bus Line
-	6700 5800 6700 5900
-Wire Bus Line
-	6700 5900 6700 6100
-Wire Bus Line
-	8150 6100 6700 6100
-Wire Bus Line
-	8150 1350 8150 1600
-Wire Bus Line
-	8150 1600 8150 1700
-Wire Bus Line
-	8150 1700 8150 1800
-Wire Bus Line
-	8150 1800 8150 1900
-Wire Bus Line
-	8150 1900 8150 2850
-Wire Bus Line
-	8150 2850 8150 3000
-Wire Bus Line
-	8150 3000 8150 3150
-Wire Bus Line
-	8150 3150 8150 3300
-Wire Bus Line
-	8150 3300 8150 3450
-Wire Bus Line
-	8150 3450 8150 3950
-Wire Bus Line
-	8150 3950 8150 4100
-Wire Bus Line
-	8150 4100 8150 4250
-Wire Bus Line
-	8150 4250 8150 4400
-Wire Bus Line
-	8150 4400 8150 4550
-Wire Bus Line
-	8150 4550 8150 4700
-Wire Bus Line
-	8150 4700 8150 4850
-Wire Bus Line
-	8150 4850 8150 5000
-Wire Bus Line
-	8150 5000 8150 5150
-Wire Bus Line
-	8150 5150 8150 5300
-Wire Bus Line
-	8150 5300 8150 5450
-Wire Bus Line
-	8150 5450 8150 5600
-Wire Bus Line
-	8150 5600 8150 5750
-Wire Bus Line
-	8150 5750 8150 5900
-Wire Bus Line
-	8150 5900 8150 6050
-Wire Bus Line
-	8150 6050 8150 6100
+	8150 6100 8150 1350
 Wire Wire Line
 	8250 3850 8900 3850
@@
 	6200 3300 6300 3400
 Wire Bus Line
-	6300 800  6300 1550
-Wire Bus Line
-	6300 1550 6300 3400
-Wire Bus Line
-	6300 3400 6300 3500
-Wire Bus Line
-	6300 3500 6300 3600
+	6300 800  6300 3600
 Wire Bus Line
 	6300 800  4350 800
 Wire Bus Line
-	4350 800  4350 1250
-Wire Bus Line
-	4350 1250 4350 1350
-Wire Bus Line
-	4350 1350 4350 2100
+	4350 800  4350 2100
 Connection ~ 3700 1550
 Text Label 4500 1550 0    60   ~ 0
@@
 F 0 "P1" H 5250 1750 50  0000 C CNN
 F 1 "ISP" V 5250 1550 40  0000 C CNN
-F 2 "" H 5250 1500 60  0000 C CNN
+F 2 "Socket_Strips:Socket_Strip_Straight_2x03" H 5250 1500 60  0001 C CNN
 F 3 "" H 5250 1500 60  0000 C CNN
 	1    5250 1500
@@
 F 0 "P2" H 9250 1900 50  0000 C CNN
 F 1 "GPIO Port" V 9300 1650 50  0000 C CNN
-F 2 "" H 9250 1650 60  0000 C CNN
+F 2 "Socket_Strips:Socket_Strip_Straight_1x04" H 9250 1650 60  0001 C CNN
 F 3 "" H 9250 1650 60  0000 C CNN
 	1    9250 1650
@@
 NoConn ~ 3050 2750
 Wire Wire Line
-	700  1050 1000 1050
-Wire Wire Line
-	1000 1050 1300 1050
-Wire Wire Line
-	1300 1050 1600 1050
-Wire Wire Line
-	1600 1050 1900 1050
+	700  1050 1900 1050
 Wire Wire Line
 	700  1050 700  1200
@@
 F 0 "C8" H 750 1500 50  0000 L CNN
 F 1 "1uF" H 750 1300 50  0000 L CNN
-F 2 "" H 700 1400 60  0000 C CNN
+F 2 "Capacitors_SMD:C_0805" H 700 1400 60  0001 C CNN
 F 3 "" H 700 1400 60  0000 C CNN
 	1    700  1400
@@
 F 0 "C4" H 1050 1500 50  0000 L CNN
 F 1 "100nF" H 1050 1300 50  0000 L CNN
-F 2 "" H 1000 1400 60  0000 C CNN
+F 2 "Capacitors_SMD:C_0805" H 1000 1400 60  0001 C CNN
 F 3 "" H 1000 1400 60  0000 C CNN
 	1    1000 1400
@@
 F 0 "C5" H 1350 1500 50  0000 L CNN
 F 1 "100nF" H 1350 1300 50  0000 L CNN
-F 2 "" H 1300 1400 60  0000 C CNN
+F 2 "Capacitors_SMD:C_0805" H 1300 1400 60  0001 C CNN
 F 3 "" H 1300 1400 60  0000 C CNN
 	1    1300 1400
@@
 $EndComp
 Wire Wire Line
-	1300 900  1300 1050
-Wire Wire Line
-	1300 1050 1300 1200
+	1300 900  1300 1200
 Connection ~ 1300 1050
 $Comp
@@
 F 0 "C6" H 1650 1500 50  0000 L CNN
 F 1 "100nF" H 1650 1300 50  0000 L CNN
-F 2 "" H 1600 1400 60  0000 C CNN
+F 2 "Capacitors_SMD:C_0805" H 1600 1400 60  0001 C CNN
 F 3 "" H 1600 1400 60  0000 C CNN
 	1    1600 1400
@@
 F 0 "C7" H 1950 1500 50  0000 L CNN
 F 1 "100nF" H 1950 1300 50  0000 L CNN
-F 2 "" H 1900 1400 60  0000 C CNN
+F 2 "Capacitors_SMD:C_0805" H 1900 1400 60  0001 C CNN
 F 3 "" H 1900 1400 60  0000 C CNN
 	1    1900 1400
@@
 	700  1600 700  1750
 Wire Wire Line
-	700  1750 1000 1750
-Wire Wire Line
-	1000 1750 1300 1750
-Wire Wire Line
-	1300 1750 1600 1750
-Wire Wire Line
-	1600 1750 1900 1750
+	700  1750 1900 1750
 Wire Wire Line
 	1000 1750 1000 1600
 Wire Wire Line
-	1300 1600 1300 1750
-Wire Wire Line
-	1300 1750 1300 1900
+	1300 1600 1300 1900
 Connection ~ 1000 1750
 Wire Wire Line
@@
 Connection ~ 1600 1750
 $Comp
-L VCC #PWR?
+L VCC #PWR020
 U 1 1 578E955E
 P 1300 900
-F 0 "#PWR?" H 1300 1000 30  0001 C CNN
+F 0 "#PWR020" H 1300 1000 30  0001 C CNN
 F 1 "VCC" H 1300 1000 30  0000 C CNN
 F 2 "" H 1300 900 60  0000 C CNN
@@
 $EndComp
 $Comp
-L GND #PWR?
+L GND #PWR021
 U 1 1 578EF284
 P 1300 1900
-F 0 "#PWR?" H 1300 1900 30  0001 C CNN
+F 0 "#PWR021" H 1300 1900 30  0001 C CNN
 F 1 "GND" H 1300 1830 30  0001 C CNN
 F 2 "" H 1300 1900 60  0000 C CNN

Commit message: a lot of changes
Connections:
- net GPIO0: no longer P2.4 (P4)
- net SCK renamed GPIO1
- net GPIO1: now also P2.4 (P4)
Changed lines of the file:
@@
 MOSI
 Text Label 6400 3500 0    60   ~ 0
-MOSI
+SCK
 Text Label 6600 3300 0    60   ~ 0
 Col6
 Text Label 6600 3400 0    60   ~ 0
 GPIO0
-Text Label 6600 3500 0    60   ~ 0
+Text Label 6050 3500 0    60   ~ 0
 GPIO1
 Text Label 6250 3700 0    60   ~ 0
@@
 Text Label 8350 1600 0    60   ~ 0
 GPIO2
+Text Label 8350 1800 0    60   ~ 0
+GPIO1
 Text Label 8350 1700 0    60   ~ 0
-GPIO1
-Text Label 8350 1800 0    60   ~ 0
 GPIO0
 $Comp

Commit message: final version
Parts:
- removed P2: GPIO Port, Socket_Strips:Socket_Strip_Straight_1x04, symbol CONN_4
- added P2: GPIO Port, symbol CONN_5
Connections:
- net GPIO0: now also P2.3
- net GPIO1: now also P2.4
- net GPIO2: now also P2.2
- net GPIO3: now also P2.1
- net GPIO4: now also P2.5
Changed lines of the file:
@@
-	1    0    0    -1
-$EndComp
-$Comp
-L CONN_4 P2
-U 1 1 578A5BB9
-P 9250 1650
-F 0 "P2" H 9250 1900 50  0000 C CNN
-F 1 "GPIO Port" V 9300 1650 50  0000 C CNN
-F 2 "Socket_Strips:Socket_Strip_Straight_1x04" H 9250 1650 60  0001 C CNN
-F 3 "" H 9250 1650 60  0000 C CNN
-	1    9250 1650
 	1    0    0    -1
 $EndComp
@@
 	1    0    0    -1
 $EndComp
+$Comp
+L CONN_5 P2
+U 1 1 577C8A1F
+P 9300 1700
+F 0 "P2" V 9250 1700 50  0000 C CNN
+F 1 "GPIO Port" V 9350 1700 50  0000 C CNN
+F 2 "" H 9300 1700 60  0000 C CNN
+F 3 "" H 9300 1700 60  0000 C CNN
+	1    9300 1700
+	1    0    0    -1
+$EndComp
+Entry Wire Line
+	8150 2000 8250 1900
+Wire Wire Line
+	8250 1900 8900 1900
+Text Label 8350 1900 0    60   ~ 0
+GPIO4
 $EndSCHEMATC
