File: keyboard.kicad_pcb (KiCad board)
At the start: 2 copper layers, 229.9 x 77.5 mm, 212 parts, among them IC1 ATMEGA32U4, J1 USBMINI_B05, P1 ISP, P2 GPIO Port, Q1 MOS_P, X1 CRYSTAL

Commit message: Update Silkscreen
Other:
- board text added: "CryptoWall40"
- board text removed: "CyptoWall40"
Changed lines of the file:
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@@
   (gr_line (start 36.322 46.736) (end 40.132 42.926) (angle 90) (layer Edge.Cuts) (width 0.15))
   (gr_line (start 36.322 116.586) (end 40.132 120.396) (angle 90) (layer Edge.Cuts) (width 0.15))
-  (gr_text "CyptoWall40\n" (at 199.39 108.712) (layer B.SilkS)
+  (gr_text "CryptoWall40\n" (at 199.39 108.712) (layer B.SilkS)
     (effects (font (size 5.08 5.08) (thickness 1.27)) (justify mirror))
   )

Commit message: Rev 1.0 Pro
Routing:
- net (no net): track 1.01 -> 0.76 mm, vias 1 -> 0
Other:
- board text added: "Rev 1.0 Pro"
- board text removed: "Rev Final"
Changed lines of the file:
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@@
     (thickness 1.6)
     (drawings 31)
-    (tracks 2711)
+    (tracks 2709)
     (zones 0)
     (modules 212)
@@
     )
   )
-  (gr_text "Rev Final\n" (at 169.926 110.998) (layer B.SilkS)
-    (effects (font (size 1.5 1.5) (thickness 0.3)) (justify mirror))
+  (gr_text "Rev 1.0 Pro" (at 169.79 111.86) (layer B.SilkS)
+    (effects (font (size 1.143 1.143) (thickness 0.28575)) (justify mirror))
   )
   (gr_text "MISO\n" (at 176.53 112.522) (layer B.SilkS)
@@
   (segment (start 234.188 98.804) (end 234.414 99.03) (width 0.25) (layer B.Cu) (net 0))
   (segment (start 234.414 101.63) (end 234.414 101.85152) (width 0.25) (layer B.Cu) (net 0))
-  (segment (start 191.516 101.6) (end 191.516 101.854) (width 0.25) (layer B.Cu) (net 0))
-  (via (at 191.516 101.6) (size 0.6) (drill 0.4) (layers F.Cu B.Cu) (net 0))
   (segment (start 151.114 57.15) (end 151.13 57.166) (width 0.25) (layer F.Cu) (net 0))
   (segment (start 139.672 60.676) (end 139.476 60.676) (width 0.25) (layer B.Cu) (net 0))
